File: Hardware/OPC/main.sch (KiCad schematic (older format))
At the start: 8 parts

Commit message: Added relay driver
Connections:
- net PEDAL_5 is gone; now on net PEDAL_4: U?.31 (A6/MISO1)
- net PEDAL_0: now also U?.27 (A2/U2TX); no longer U?.26 (A1)
- net PEDAL_1: now also U?.28 (A3/U2RX); no longer U?.27 (A2/U2TX)
- net PEDAL_2: now also U?.29 (A4/NSS1); no longer U?.28 (A3/U2RX)
- net PEDAL_3: now also U?.30 (A5/SCK1); no longer U?.29 (A4/NSS1)
- net PEDAL_4: no longer U?.30 (A5/SCK1)
- new net TUNER: U?.26 (A1)
Changed lines of the file:
@@
 Text HLabel 3200 7350 2    50   Output ~ 0
 GND
-Text HLabel 9800 3650 2    50   Output ~ 0
+Text HLabel 9800 3500 2    50   Output ~ 0
 PEDAL_0
-Text HLabel 9800 3500 2    50   Output ~ 0
+Text HLabel 9800 3350 2    50   Output ~ 0
 PEDAL_1
-Text HLabel 9800 3350 2    50   Output ~ 0
+Text HLabel 9800 3200 2    50   Output ~ 0
 PEDAL_2
-Text HLabel 9800 3200 2    50   Output ~ 0
+Text HLabel 9800 3050 2    50   Output ~ 0
 PEDAL_3
-Text HLabel 9800 3050 2    50   Output ~ 0
+Text HLabel 9800 2900 2    50   Output ~ 0
 PEDAL_4
-Text HLabel 9800 2900 2    50   Output ~ 0
-PEDAL_5
 Wire Wire Line
 	9800 2900 9750 2900
@@
 Wire Wire Line
 	9750 3650 9800 3650
+Text HLabel 9800 3650 2    50   Output ~ 0
+TUNER
 $EndSCHEMATC

Commit message: Added 7 seg display
Connections:
- net 7SEG_A: now reaches U?.1 (B12/NSS2)
- net 7SEG_B: now reaches U?.2 (B13/SCK2)
- net 7SEG_C: now reaches U?.3 (B14/MISO2)
- net 7SEG_D: now reaches U?.4 (B15/MOSI2)
- net 7SEG_E: now reaches U?.5 (A8/MCO)
- net 7SEG_F: now reaches U?.6 (A9/U1TXa)
- net 7SEG_G: now reaches U?.7 (A10/U1RXa)
Changed lines of the file:
@@
 $Descr A4 11693 8268
 encoding utf-8
-Sheet 2 3
+Sheet 2 4
 Title ""
 Date ""
@@
 Text HLabel 9800 3650 2    50   Output ~ 0
 TUNER
+Text HLabel 7600 1550 0    50   Output ~ 0
+7SEG_A
+Text HLabel 7600 1700 0    50   Output ~ 0
+7SEG_B
+Text HLabel 7600 1850 0    50   Output ~ 0
+7SEG_C
+Text HLabel 7600 2000 0    50   Output ~ 0
+7SEG_D
+Text HLabel 7600 2300 0    50   Output ~ 0
+7SEG_F
+Text HLabel 7600 2450 0    50   Output ~ 0
+7SEG_G
+Text HLabel 7600 2150 0    50   Output ~ 0
+7SEG_E
+Wire Wire Line
+	7600 1550 7650 1550
+Wire Wire Line
+	7600 1700 7650 1700
+Wire Wire Line
+	7650 1850 7600 1850
+Wire Wire Line
+	7600 2000 7650 2000
+Wire Wire Line
+	7650 2150 7600 2150
+Wire Wire Line
+	7650 2300 7600 2300
+Wire Wire Line
+	7650 2450 7600 2450
 $EndSCHEMATC
